Commit message: new files for arm control

File: squirtle_manipulator/squirtle_arm_description/urdf/arm.urdf.xacro (robot description, xacro)
@@ -15,5 +15,5 @@
       <!-- Place the "floating" arm at the location it should be if mounted on a turtlebot,
            as pick and place and other demos assume this location -->
-      <origin xyz="0.06 0.00 0.762" rpy="0 0 0" />
+      <origin xyz="0.06 0.00 0.762" rpy="0 1.5708 0" />
     </turtlebot_arm>
 </robot>
